Commit message: Add files via upload

File: scout_mini_ros2/scout_mini_description/urdf/scout_mini.urdf.xacro (robot description, xacro)
@@ -26,5 +26,5 @@
     <parent link="base_link" />
     <child link="camera_link"/>
-    <origin xyz="0.185 0 0.15" rpy="0 0 0"/>
+    <origin xyz="-0.035 0 0.52" rpy="0 0 0"/>
   </joint>
   <joint name="inertial_joint" type="fixed">
